File: examples/harness-box/harness-box.kicad_sch (KiCad schematic)
At the start: 18 parts, among them CN1 212528-0400, Q1 DMN3200U-7, U1 5018761840, U2 DG419LEDY-T1-GE4, U3 DG419LEDY-T1-GE4, U4 SMF16A, U5 STPS2H100ZFY

Commit message: Clean up ts-kicad and complete the harness-box example
Parts:
- Q1: symbol overrides:C461018__DMN3200U-7__a74af1ae -> C461018:DMN3200U-7
- R1, R2, R3, R4, R5, R6, R7, R8: footprint C21190:R0603 -> Resistor_SMD:R_0603_1608Metric
- U2, U3: symbol overrides:C2673265__DG419LEDY-T1-GE4__7dbfe9aa -> C2673265:DG419LEDY-T1-GE4
